File: Battery Controller.sch (KiCad schematic (older format))
At the start: 27 parts, among them Q17 ZXMP10A13FTA, Q18 Q_NMOS_DGS, SW2 SW_Push, U3 BQ78350-R1

Commit message: Good-enough for first PCB attempt.
Parts:
- added R7, R8: 100k, Resistor_SMD:R_0603_1608Metric, symbol bldc-BMS-rescue:R_Small
- C28, C30, C31: Description (none) -> CAP CER 0.1UF 25V X7R 0603; Digikey PN (none) -> 311-1341-1-ND
- C29: Description (none) -> CAP CER 3.3UF 10V X5R 0805; Digikey PN (none) -> 1276-2912-1-ND
- D23, D24, D25, D26, D27: Description (none) -> LED GREEN CLEAR 0603 SMD; Digikey PN (none) -> 732-4971-1-ND
- Q17: footprint (none) -> Package_TO_SOT_SMD:SOT-23; Description (none) -> MOSFET P-CH 100V 0.6A SOT23-3; Digikey PN (none) -> ZXMP10A13FCT-ND
- Q18: value Q_NMOS_DGS -> Q_NMOS_GSD; footprint (none) -> Package_TO_SOT_SMD:SOT-23; symbol bldc-BMS-rescue:Q_NMOS_DGS -> Device:Q_NMOS_GSD; Description (none) -> MOSFET N-CH 20V 0.63A SOT23-3; Digikey PN (none) -> DMN2004KDICT-ND
- R69, R70: value 510k -> 100k
- SW2: footprint (none) -> Button_Switch_SMD:SW_SPST_PTS810; Description (none) -> SWITCH TACTILE SPST-NO 50MA 32V; Digikey PN (none) -> CKN10684CT-ND
- U3: symbol bldc-BMS-rescue:BQ78350 -> bldc-BMS-rescue:BQ78350-bldc-BMS-rescue; Description (none) -> IC BATTERY MGMT CTRLR 30TSSOP; Digikey PN (none) -> 296-44315-1-ND
Connections:
- net GND: now also Q18.2 (S); no longer Q18.3 (S)
- net PMON_EN: now also Q18.1 (G); no longer Q18.2 (G)
- net REGOUT: now also R7.1, R8.1
- net SDA: now also R7.2
- net at R61.2: now also Q18.3 (D); no longer Q18.1 (D)
- net SDL renamed SCL
- net SCL: now also R8.2
Other:
- note added: "~PRES\n- Use as master ON/OFF\n- If high for 4x 250ms samples, CHG, DSG AND PCHG FETs are disabled.\n- If low, system can enable."
- note removed: "Need 10mA from 20V:\nV=IR; R=V/I = 20V/10mA = 2k"
- note removed: "~PRES\n- If high for 4x 250ms samples, CHG, DSG AND PCHG FETs are disabled.\n- If low, system can enable."
- moved on the sheet: C28, C29, Q17, Q18, R58, R59, R60, R61
