File: bldc-BMS.sch (KiCad schematic (older format))
At the start: 7 parts

Commit message: Updated top-level connections and added MCU
Parts:
- removed J? (x2): Conn_01x01, symbol Conn_01x01
- removed U?: BQ78350, TSSOP-30, symbol BQ78350
- removed U?: STM32F072C8Tx, Housings_QFP:LQFP-48_7x7mm_Pitch0.5mm, symbol STM32F072C8Tx
- removed U?: bq76930, symbol bq76930
- added F1: 100mA, Fuse:Fuse_0805_2012Metric, symbol Device:Polyfuse
- added J1, J5: Conn_01x04, Connector_JST:JST_PH_B4B-PH-K_1x04_P2.00mm_Vertical, symbol bldc-BMS-rescue:Conn_01x04
- added J10: USB_B_Micro, Connector_USB:USB_Micro-B_Molex_47346-0001, symbol Connector:USB_B_Micro
- added J2: Conn_01x07, Connector_JST:JST_PH_B7B-PH-K_1x07_P2.00mm_Vertical, symbol Connector_Generic:Conn_01x07
- added J8: Conn_01x06, Connector_JST:JST_PH_B6B-PH-K_1x06_P2.00mm_Vertical, symbol Connector_Generic:Conn_01x06
- added J9: Conn_01x02, Connector_JST:JST_PH_B3B-PH-K_1x03_P2.00mm_Vertical, symbol bldc-BMS-rescue:Conn_01x02
- J3, J6: renamed from J?; value Conn_01x01 -> Conn_01x02; footprint (none) -> bldc-BMS:XT60PW-F; symbol Conn_01x01 -> bldc-BMS-rescue:Conn_01x02
Connections:
- net labels added: GND
- net labels removed: +BATT, +VDC, -BATT, -VDC
- wire segments 8 -> 93
Other:
- note added: "6 Cell Configuration\nC2 == C4\nC7 == C9"
- note added: "AMASS XT60PW?\nhttps://www.tme.eu/gb/details/xt60pw-f/dc-power-connectors/amass/"
- note added: "CELL 6\nCELL 5\nCELL 4\nCELL 3\nCELL 2\nCELL 1"
- note added: "SYSTEM ENABLE\nLATCH"

Commit message: Good-enough for first PCB attempt.
Parts:
- added JP1: Jumper_NO, Jumper:SolderJumper-2_P1.3mm_Open_TrianglePad1.0x1.5mm, symbol Device:Jumper_NO_Small
- added NT1: Net-Tie, NetTie:NetTie-2_SMD_Pad0.5mm, symbol Device:Net-Tie_2
- added TP1: SCL, TestPoint:TestPoint_Pad_D1.5mm, symbol Connector:TestPoint
- added TP10: BAT-, TestPoint:TestPoint_Pad_D1.5mm, symbol Connector:TestPoint
- added TP2: SMBC, TestPoint:TestPoint_Pad_D1.5mm, symbol Connector:TestPoint
- added TP3: REGOUT, TestPoint:TestPoint_Pad_D1.5mm, symbol Connector:TestPoint
- added TP4: SDA, TestPoint:TestPoint_Pad_D1.5mm, symbol Connector:TestPoint
- added TP5: SMBD, TestPoint:TestPoint_Pad_D1.5mm, symbol Connector:TestPoint
- added TP6: BAT+, TestPoint:TestPoint_Pad_D1.5mm, symbol Connector:TestPoint
- added TP7: LOAD+, TestPoint:TestPoint_Pad_D1.5mm, symbol Connector:TestPoint
- added TP8: 3.3V, TestPoint:TestPoint_Pad_D1.5mm, symbol Connector:TestPoint
- added TP9: 5V, TestPoint:TestPoint_Pad_D1.5mm, symbol Connector:TestPoint
- F1: Description (none) -> PTC RESET FUSE 15V 50MA 0603; Digikey PN (none) -> 507-1816-1-ND
- J1, J5: footprint Connector_JST:JST_PH_B4B-PH-K_1x04_P2.00mm_Vertical -> Connector_JST:JST_PH_S4B-PH-K_1x04_P2.00mm_Horizontal; Description (none) -> CONN HEADER R/A 4POS 2MM; Digikey PN (none) -> 455-1721-ND
- J10: footprint Connector_USB:USB_Micro-B_Molex_47346-0001 -> bldc-BMS:USB_Micro-B_Amphenol_10103594-0001LF_Horizontal_circular; Description (none) -> CONN RCPT USB2.0 MICRO B SMD R/A; Digikey PN (none) -> 609-4050-1-ND
- J2: footprint Connector_JST:JST_PH_B7B-PH-K_1x07_P2.00mm_Vertical -> Connector_JST:JST_PH_S7B-PH-K_1x07_P2.00mm_Horizontal; Description JST PH 2mm 7pin -> CONN HEADER R/A 7POS 2MM; Digikey PN (none) -> 455-1724-ND
- J3: value Conn_01x02 -> XT60_MALE; footprint bldc-BMS:XT60PW-F -> bldc-BMS:XT60PW-M20; symbol bldc-BMS-rescue:Conn_01x02 -> bldc-BMS:XT60_male
- J6: value Conn_01x02 -> XT60_FEMALE; footprint bldc-BMS:XT60PW-F -> bldc-BMS:XT60PW-F20; symbol bldc-BMS-rescue:Conn_01x02 -> bldc-BMS:XT60_female
- J8: footprint Connector_JST:JST_PH_B6B-PH-K_1x06_P2.00mm_Vertical -> Connector_JST:JST_PH_S6B-PH-K_1x06_P2.00mm_Horizontal; Description JST PH 2mm 6pin -> CONN HEADER R/A 6POS 2MM; Digikey PN (none) -> 455-1723-ND
- J9: footprint Connector_JST:JST_PH_B3B-PH-K_1x03_P2.00mm_Vertical -> Connector_JST:JST_PH_S2B-PH-K_1x02_P2.00mm_Horizontal; Description (none) -> CONN HEADER R/A 2POS 2MM; Digikey PN (none) -> 455-1719-ND
Connections:
- net Battery Controller/C10: now also J2.1 (Pin_1), TP3.1; no longer J2.7 (Pin_7)
- net Battery Controller/SDA: now also TP4.1
- net Battery Controller/SMBC: now also TP2.1
- net Battery Controller/SMBD: now also TP5.1
- net Battery Monitor/C0: now also J2.7 (Pin_7); no longer J2.1 (Pin_1)
- net Battery Monitor/C1: now also J2.6 (Pin_6); no longer J2.2 (Pin_2)
- net Battery Monitor/C2: now also J2.5 (Pin_5); no longer J2.3 (Pin_3)
- net Battery Monitor/C6: now also J2.3 (Pin_3); no longer J2.5 (Pin_5)
- net Battery Monitor/C7: now also J2.2 (Pin_2); no longer J2.6 (Pin_6)
- net Battery Monitor/LOAD+: now also TP7.1
- net CAN and USB Interface/3.3V: now also TP8.1
- net GND: now also NT1.2; no longer J3.1 (Pin_1)
- net Power Stage/BAT+: now also J3.1 (POS), TP6.1; no longer J3.2 (Pin_2)
- net at J10.1 (VBUS): now also JP1.2
- new net Battery Controller/SCL: TP1.1
- new net CAN and USB Interface/+5V: JP1.1, TP9.1
- new net Power Stage/BAT-: J3.2 (NEG), NT1.1, TP10.1
- no-connect marks 0 -> 3
Other:
- note added: "BATTERY TEMPERATURE SENSORS\n10kOHM NTC"
- note added: "CAN"
- note added: "Notes:\n- 25V maximum\n- 20A discharge\n- ??A charge"
- note added: "SWD PROGRAMMING"
- note added: "SYSTEM ENABLE\nPIN1+2: ENABLE SWITCH\nPIN3+4: LED ON OUTPUT"
- note added: "TO BATTERY"
- note added: "TO LOAD/CHARGER"
- note removed: "6 Cell Configuration\nC2 == C4\nC7 == C9"
- note removed: "SYSTEM ENABLE\nLATCH"
