File: power_stage.sch (KiCad schematic (older format))
At the start: 23 parts

Commit message: Updated top-level connections and added MCU
Parts:
- removed D?: MURS360T3G, symbol D_ALT
- removed Q?: ZXMP10A13FTA, symbol Q_PMOS_DGS
- removed Q? (x2): TBC, symbol Q_NMOS_DGS
- removed R?: 1M, symbol R
- removed R?: 1k, symbol R
- added C2: 1uF, Capacitor_SMD:C_0603_1608Metric, symbol bldc-BMS-rescue:C
- added C5: 0.01uF, Capacitor_SMD:C_0603_1608Metric, symbol bldc-BMS-rescue:C
- added D2, D3: 3.3V, Diode_SMD:D_0603_1608Metric, symbol bldc-BMS-rescue:D_Schottky_ALT
- added D5: GREEN, LED_SMD:LED_0603_1608Metric_Pad1.05x0.95mm_HandSolder, symbol Device:LED_ALT
- added Q5: Q_PMOS_DGS, symbol Device:Q_PMOS_DGS
- added R1, R16: 100R, Resistor_SMD:R_0603_1608Metric, symbol bldc-BMS-rescue:R
- added R11: 2k, Resistor_SMD:R_0603_1608Metric, symbol bldc-BMS-rescue:R_Small
- added R12, R13, R14: 1k, Resistor_SMD:R_0603_1608Metric, symbol bldc-BMS-rescue:R
- added R15, R6, R9: 220R, Resistor_SMD:R_0603_1608Metric, symbol bldc-BMS-rescue:R
- added U1: bq76200, Package_SO:HTSSOP-28-1EP_4.4x9.7mm_P0.65mm_EP3.4x9.5mm_ThermalVias, symbol bldc-BMS:bq76200
- C1, C3, C4, C6, C7, C8, C9: renamed from C?; footprint (none) -> Capacitor_SMD:C_0603_1608Metric; symbol C -> bldc-BMS-rescue:C
- D1: renamed from D?; footprint (none) -> Diode_SMD:D_SMC; symbol D_Schottky_ALT -> bldc-BMS-rescue:D_Schottky_ALT
- D4: renamed from D?; footprint (none) -> Diode_SMD:D_0603_1608Metric; symbol D_Schottky_ALT -> bldc-BMS-rescue:D_Schottky_ALT
- D6: renamed from D?; symbol D_ALT -> bldc-BMS-rescue:D_ALT
- Q2, Q3: renamed from Q?; footprint (none) -> Package_SO:PowerPAK_SO-8_Single; symbol Q_NMOS_DGS -> bldc-BMS-rescue:Q_NMOS_DGS
- R10, R5: renamed from R?; footprint (none) -> Resistor_SMD:R_0603_1608Metric; symbol R -> bldc-BMS-rescue:R
- R2, R4: renamed from R?; value 100 -> 100R; footprint (none) -> Resistor_SMD:R_0603_1608Metric; symbol R -> bldc-BMS-rescue:R
- R3: renamed from R?; value 0.001R -> 0.005R; footprint (none) -> Resistor_SMD:R_2816_7142Metric; symbol R -> bldc-BMS-rescue:R
Connections:
- net labels added: BAT+, BAT-, CP_EN, LOAD+, LOAD-, PCHG, PMON_EN
- net labels removed: +BATT, +VDC, -BATT, -VDC, C0, PFD
- wire segments 64 -> 110
Other:
- note added: "Sense Resistor:\nSPR-SRN max is 300mV\nRsense = 300mV / 20A = 0.012Ohm; need half (7.5mOhm)\nP=I^2R = 20^2*0.005 = 2W\n"
- note removed: "Section purpose?"
- note removed: "Sense Resistor:\n0.001Ohm (1mOhm)\nSense Range: +/-?A\nP=I^2R = 50^2*0.001 = 2.5W\nLSB = ??mA"
- note removed: "TODO: Add pre-charge circuit!"
- moved on the sheet: R10, R3

Commit message: Good-enough for first PCB attempt.
Parts:
- C1, C3, C4, C6, C7, C8, C9: Description (none) -> CAP CER 0.1UF 25V X7R 0603; Digikey PN (none) -> 311-1341-1-ND
- C2: value 1uF -> 1uF 10V; Description (none) -> CAP CER 1UF 25V X5R 0603; Digikey PN (none) -> 1276-1102-1-ND
- C5: Description (none) -> CAP CER 10000PF 50V X7R 0603; Digikey PN (none) -> 1276-1921-1-ND
- D1: Description (none) -> TVS DIODE 45V 72.7V DO214AB; Digikey PN (none) -> SMCJ45ALFCT-ND
- D2, D3: footprint Diode_SMD:D_0603_1608Metric -> Diode_SMD:D_SOD-323; Description (none) -> TVS DIODE 3.3V SOD323; Digikey PN (none) -> 1727-4152-1-ND
- D4: footprint Diode_SMD:D_0603_1608Metric -> Diode_SMD:D_SOD-123; Description (none) -> DIODE ZENER 16V 500MW SOD123; Digikey PN (none) -> MMSZ5246B-FDICT-ND
- D5: Description (none) -> LED GREEN CLEAR 0603 SMD; Digikey PN (none) -> 732-4971-1-ND
- D6: footprint (none) -> Diode_SMD:D_SMC; Description (none) -> DIODE GEN PURP 600V 3A SMC; Digikey PN (none) -> MURS360T3GOSCT-ND
- Q2, Q3: value TBC -> CSD18531Q5A; footprint Package_SO:PowerPAK_SO-8_Single -> Package_TO_SOT_SMD:TDSON-8-1; symbol bldc-BMS-rescue:Q_NMOS_DGS -> Transistor_FET:CSD18531Q5A; Description (none) -> MOSFET N-CH 60V 8SON 4.6mOHM; Digikey PN (none) -> 296-30573-1-ND
- Q5: value Q_PMOS_DGS -> Q_PMOS; footprint (none) -> Package_TO_SOT_SMD:SOT-23-6; symbol Device:Q_PMOS_DGS -> bldc-BMS:Q_PMOS_6pin; Description (none) -> MOSFET P-CH 60V 4A CPH6; Digikey PN (none) -> CPH6354-TL-WOSCT-ND
- R12, R13, R14: footprint Resistor_SMD:R_0603_1608Metric -> Resistor_SMD:R_1206_3216Metric; Description (none) -> RES SMD 1K OHM 5% 1/4W 1206; Digikey PN (none) -> 311-1.0KERCT-ND
- R3: footprint Resistor_SMD:R_2816_7142Metric -> Resistor_SMD:R_2512_6332Metric_Pad1.52x3.35mm_HandSolder; Description (none) -> RES 0.005 OHM 1% 3W 2512; Digikey PN (none) -> CRE2512-FZ-R005E-3CT-ND
- U1: footprint Package_SO:HTSSOP-28-1EP_4.4x9.7mm_P0.65mm_EP3.4x9.5mm_ThermalVias -> Package_SO:TSSOP-16_4.4x5mm_P0.65mm; Description (none) -> HIGH-SIDE N-CH FET DRVR 16TSSOP; Digikey PN (none) -> 296-43273-1-ND
Connections:
- net BAT+: now also Q2.1 (S), Q2.2 (S)
- net LOAD+: now also Q3.1 (S), Q3.2 (S), Q5.2 (D), Q5.5 (D), Q5.6 (D)
- net at R12.2, R13.2, R14.2: now also Q2.5 (D), Q3.5 (D); no longer Q2.1 (D), Q3.1 (D)
- net at R6.2: now also Q2.4 (G); no longer Q2.2 (G)
- net at R9.2: now also Q3.4 (G); no longer Q3.2 (G)
- net at R12.1, R13.1, R14.1: now also Q5.4 (S); no longer Q5.3 (S)
- net at R15.2: now also Q5.3 (G); no longer Q5.2 (G)
Other:
- note added: "Sense Resistor:\nSRP-SRN max is 300mV\nRsense = 300mV / 20A = 0.012Ohm; need half (7.5mOhm)\nP=I^2R = 20^2*0.005 = 2W\n"
- note removed: "Sense Resistor:\nSPR-SRN max is 300mV\nRsense = 300mV / 20A = 0.012Ohm; need half (7.5mOhm)\nP=I^2R = 20^2*0.005 = 2W\n"
Changed lines of the file:
@@
 EESchema Schematic File Version 4
 LIBS:bldc-BMS-cache
-EELAYER 26 0
+EELAYER 29 0
 EELAYER END
 $Descr A4 11693 8268
 encoding utf-8
 Sheet 2 5
-Title ""
-Date ""
-Rev ""
+Title "bldc-BMS"
+Date "2018-09-02"
+Rev "1.0"
 Comp ""
 Comment1 ""
@@
 F 2 "Diode_SMD:D_SMC" H 1650 5600 50  0001 C CNN
 F 3 "" H 1650 5600 50  0001 C CNN
+F 4 "TVS DIODE 45V 72.7V DO214AB" H 0   0   50  0001 C CNN "Description"
+F 5 "SMCJ45ALFCT-ND" H 0   0   50  0001 C CNN "Digikey PN"
 	1    1650 5600
 	0    1    1    0
@@
 $EndComp
 $Comp
-L bldc-BMS-rescue:Q_NMOS_DGS Q2
+L Transistor_FET:CSD18531Q5A Q2
 U 1 1 5B1D5D28
 P 4700 5000
-F 0 "Q2" H 4900 5050 50  0000 L CNN
-F 1 "TBC" H 4900 4950 50  0000 L CNN
-F 2 "Package_SO:PowerPAK_SO-8_Single" H 4900 5100 50  0001 C CNN
+F 0 "Q2" V 4550 5150 50  0000 L CNN
+F 1 "CSD18531Q5A" V 5000 4950 50  0000 L CNN
+F 2 "Package_TO_SOT_SMD:TDSON-8-1" H 4900 5100 50  0001 C CNN
 F 3 "" H 4700 5000 50  0001 C CNN
+F 4 " MOSFET N-CH 60V 8SON 4.6mOHM" H 0   0   50  0001 C CNN "Description"
+F 5 "296-30573-1-ND" H 0   0   50  0001 C CNN "Digikey PN"
 	1    4700 5000
 	0    1    1    0
 $EndComp
 $Comp
-L bldc-BMS-rescue:Q_NMOS_DGS Q3
+L Transistor_FET:CSD18531Q5A Q3
 U 1 1 5B1D5E05
 P 6600 5000
-F 0 "Q3" H 6800 5050 50  0000 L CNN
-F 1 "TBC" H 6800 4950 50  0000 L CNN
-F 2 "Package_SO:PowerPAK_SO-8_Single" H 6800 5100 50  0001 C CNN
+F 0 "Q3" V 6500 5150 50  0000 L CNN
+F 1 "CSD18531Q5A" V 6900 4950 50  0000 L CNN
+F 2 "Package_TO_SOT_SMD:TDSON-8-1" H 6800 5100 50  0001 C CNN
 F 3 "" H 6600 5000 50  0001 C CNN
+F 4 " MOSFET N-CH 60V 8SON 4.6mOHM" H 0   0   50  0001 C CNN "Description"
+F 5 "296-30573-1-ND" H 0   0   50  0001 C CNN "Digikey PN"
 	1    6600 5000
 	0    -1   1    0
@@
 F 2 "Capacitor_SMD:C_0603_1608Metric" H 9138 5200 50  0001 C CNN
 F 3 "" H 9100 5350 50  0001 C CNN
+F 4 "CAP CER 0.1UF 25V X7R 0603" H 0   0   50  0001 C CNN "Description"
+F 5 "311-1341-1-ND" H 0   0   50  0001 C CNN "Digikey PN"
 	1    9100 5350
 	1    0    0    -1
@@
 F 2 "Capacitor_SMD:C_0603_1608Metric" H 9138 5550 50  0001 C CNN
 F 3 "" H 9100 5700 50  0001 C CNN
+F 4 "CAP CER 0.1UF 25V X7R 0603" H 0   0   50  0001 C CNN "Description"
+F 5 "311-1341-1-ND" H 0   0   50  0001 C CNN "Digikey PN"
 	1    9100 5700
 	1    0    0    -1
@@
 F 0 "D6" H 8500 5700 50  0000 C CNN
 F 1 "MURS360T3G" H 8500 5500 50  0000 C CNN
-F 2 "" H 8500 5600 50  0001 C CNN
+F 2 "Diode_SMD:D_SMC" H 8500 5600 50  0001 C CNN
 F 3 "" H 8500 5600 50  0001 C CNN
+F 4 "DIODE GEN PURP 600V 3A SMC" H 0   0   50  0001 C CNN "Description"
+F 5 "MURS360T3GOSCT-ND" H 0   0   50  0001 C CNN "Digikey PN"
 	1    8500 5600
 	0    1    1    0
@@
 F 0 "R3" V 3150 6100 50  0000 C CNN
 F 1 "0.005R" V 2950 6100 50  0000 C CNN
-F 2 "Resistor_SMD:R_2816_7142Metric" V 2980 6100 50  0001 C CNN
+F 2 "Resistor_SMD:R_2512_6332Metric_Pad1.52x3.35mm_HandSolder" V 2980 6100 50  0001 C CNN
 F 3 "WSHM28185L000FEA" H 3050 6100 50  0001 C CNN
+F 4 "RES 0.005 OHM 1% 3W 2512" H 0   0   50  0001 C CNN "Description"
+F 5 "CRE2512-FZ-R005E-3CT-ND" H 0   0   50  0001 C CNN "Digikey PN"
 	1    3050 6100
 	0    -1   -1   0
@@
 F 2 "Capacitor_SMD:C_0603_1608Metric" H 3088 3800 50  0001 C CNN
 F 3 "" H 3050 3950 50  0001 C CNN
+F 4 "CAP CER 0.1UF 25V X7R 0603" H 0   0   50  0001 C CNN "Description"
+F 5 "311-1341-1-ND" H 0   0   50  0001 C CNN "Digikey PN"
 	1    3050 3950
 	0    1    1    0
@@
 F 2 "Capacitor_SMD:C_0603_1608Metric" H 3588 4300 50  0001 C CNN
 F 3 "" H 3550 4450 50  0001 C CNN
+F 4 "CAP CER 0.1UF 25V X7R 0603" H 0   0   50  0001 C CNN "Description"
+F 5 "311-1341-1-ND" H 0   0   50  0001 C CNN "Digikey PN"
 	1    3550 4450
 	1    0    0    -1
@@
 F 2 "Capacitor_SMD:C_0603_1608Metric" H 2538 4300 50  0001 C CNN
 F 3 "" H 2500 4450 50  0001 C CNN
+F 4 "CAP CER 0.1UF 25V X7R 0603" H 0   0   50  0001 C CNN "Description"
+F 5 "311-1341-1-ND" H 0   0   50  0001 C CNN "Digikey PN"
 	1    2500 4450
 	1    0    0    -1
@@
 F 2 "Capacitor_SMD:C_0603_1608Metric" H 5388 5500 50  0001 C CNN
 F 3 "" H 5350 5650 50  0001 C CNN
+F 4 "CAP CER 0.1UF 25V X7R 0603" H 0   0   50  0001 C CNN "Description"
+F 5 "311-1341-1-ND" H 0   0   50  0001 C CNN "Digikey PN"
 	1    5350 5650
 	0    1    1    0
@@
 F 2 "Capacitor_SMD:C_0603_1608Metric" H 5788 5500 50  0001 C CNN
 F 3 "" H 5750 5650 50  0001 C CNN
+F 4 "CAP CER 0.1UF 25V X7R 0603" H 0   0   50  0001 C CNN "Description"
+F 5 "311-1341-1-ND" H 0   0   50  0001 C CNN "Digikey PN"
 	1    5750 5650
 	0    1    1    0
@@
 F 0 "D4" H 7350 4450 50  0000 C CNN
 F 1 "MMSZ5246B-7-F" H 7350 4250 50  0000 C CNN
-F 2 "Diode_SMD:D_0603_1608Metric" H 7350 4350 50  0001 C CNN
+F 2 "Diode_SMD:D_SOD-123" H 7350 4350 50  0001 C CNN
 F 3 "" H 7350 4350 50  0001 C CNN
+F 4 "DIODE ZENER 16V 500MW SOD123" H 0   0   50  0001 C CNN "Description"
+F 5 "MMSZ5246B-FDICT-ND" H 0   0   50  0001 C CNN "Digikey PN"
 	1    7350 4350
 	0    1    1    0
@@
 Connection ~ 7350 5100
 Text Notes 700  1100 0    60   ~ 0
-Sense Resistor:\nSPR-SRN max is 300mV\nRsense = 300mV / 20A = 0.012Ohm; need half (7.5mOhm)\nP=I^2R = 20^2*0.005 = 2W\n
+Sense Resistor:\nSRP-SRN max is 300mV\nRsense = 300mV / 20A = 0.012Ohm; need half (7.5mOhm)\nP=I^2R = 20^2*0.005 = 2W\n
 $Comp
 L bldc-BMS-rescue:D_Schottky_ALT D2
@@
 F 0 "D2" H 2200 4550 50  0000 C CNN
 F 1 "3.3V" H 2200 4350 50  0000 C CNN
-F 2 "Diode_SMD:D_0603_1608Metric" H 2200 4450 50  0001 C CNN
+F 2 "Diode_SMD:D_SOD-323" H 2200 4450 50  0001 C CNN
 F 3 "" H 2200 4450 50  0001 C CNN
+F 4 "TVS DIODE 3.3V SOD323" H 0   0   50  0001 C CNN "Description"
+F 5 "1727-4152-1-ND" H 0   0   50  0001 C CNN "Digikey PN"
 	1    2200 4450
 	0    1    1    0
@@
 F 0 "D3" H 3950 4550 50  0000 C CNN
 F 1 "3.3V" H 3950 4350 50  0000 C CNN
-F 2 "Diode_SMD:D_0603_1608Metric" H 3950 4450 50  0001 C CNN
+F 2 "Diode_SMD:D_SOD-323" H 3950 4450 50  0001 C CNN
 F 3 "" H 3950 4450 50  0001 C CNN
+F 4 "TVS DIODE 3.3V SOD323" H 0   0   50  0001 C CNN "Description"
+F 5 "1727-4152-1-ND" H 0   0   50  0001 C CNN "Digikey PN"
 	1    3950 4450
 	0    1    1    0
@@
 F 0 "R12" V 8180 3050 50  0000 C CNN
 F 1 "1k" V 8100 3050 50  0000 C CNN
-F 2 "Resistor_SMD:R_0603_1608Metric" V 8030 3050 50  0001 C CNN
+F 2 "Resistor_SMD:R_1206_3216Metric" V 8030 3050 50  0001 C CNN
 F 3 "" H 8100 3050 50  0001 C CNN
+F 4 "RES SMD 1K OHM 5% 1/4W 1206" H 8100 3050 50  0001 C CNN "Description"
+F 5 "311-1.0KERCT-ND" H 8100 3050 50  0001 C CNN "Digikey PN"
 	1    8100 3050
 	0    1    1    0
@@
 F 0 "R13" V 8180 3250 50  0000 C CNN
 F 1 "1k" V 8100 3250 50  0000 C CNN
-F 2 "Resistor_SMD:R_0603_1608Metric" V 8030 3250 50  0001 C CNN
+F 2 "Resistor_SMD:R_1206_3216Metric" V 8030 3250 50  0001 C CNN
 F 3 "" H 8100 3250 50  0001 C CNN
+F 4 "RES SMD 1K OHM 5% 1/4W 1206" H 8100 3250 50  0001 C CNN "Description"
+F 5 "311-1.0KERCT-ND" H 8100 3250 50  0001 C CNN "Digikey PN"
 	1    8100 3250
 	0    1    1    0
@@
 F 0 "R14" V 8180 3450 50  0000 C CNN
 F 1 "1k" V 8100 3450 50  0000 C CNN
-F 2 "Resistor_SMD:R_0603_1608Metric" V 8030 3450 50  0001 C CNN
+F 2 "Resistor_SMD:R_1206_3216Metric" V 8030 3450 50  0001 C CNN
 F 3 "" H 8100 3450 50  0001 C CNN
+F 4 "RES SMD 1K OHM 5% 1/4W 1206" H 8100 3450 50  0001 C CNN "Description"
+F 5 "311-1.0KERCT-ND" H 8100 3450 50  0001 C CNN "Digikey PN"
 	1    8100 3450
 	0    1    1    0
@@
 F 0 "U1" H 3550 2937 60  0000 C CNN
 F 1 "bq76200" H 3550 2831 60  0000 C CNN
-F 2 "Package_SO:HTSSOP-28-1EP_4.4x9.7mm_P0.65mm_EP3.4x9.5mm_ThermalVias" H 3550 2100 60  0001 C CNN
+F 2 "Package_SO:TSSOP-16_4.4x5mm_P0.65mm" H 3550 2100 60  0001 C CNN
 F 3 "" H 3550 2100 60  0001 C CNN
+F 4 "HIGH-SIDE N-CH FET DRVR 16TSSOP" H 0   0   50  0001 C CNN "Description"
+F 5 "296-43273-1-ND" H 0   0   50  0001 C CNN "Digikey PN"
 	1    3550 2100
 	1    0    0    -1
@@
 P 2600 1350
 F 0 "C2" H 2625 1450 50  0000 L CNN
-F 1 "1uF" H 2625 1250 50  0000 L CNN
+F 1 "1uF 10V" H 2625 1250 50  0000 L CNN
 F 2 "Capacitor_SMD:C_0603_1608Metric" H 2638 1200 50  0001 C CNN
 F 3 "" H 2600 1350 50  0001 C CNN
+F 4 "CAP CER 1UF 25V X5R 0603" H 0   0   50  0001 C CNN "Description"
+F 5 "1276-1102-1-ND" H 0   0   50  0001 C CNN "Digikey PN"
 	1    2600 1350
 	-1   0    0    -1
@@
 F 2 "Capacitor_SMD:C_0603_1608Metric" H 5188 2200 50  0001 C CNN
 F 3 "" H 5150 2350 50  0001 C CNN
+F 4 "CAP CER 10000PF 50V X7R 0603" H 0   0   50  0001 C CNN "Description"
+F 5 "1276-1921-1-ND" H 0   0   50  0001 C CNN "Digikey PN"
 	1    5150 2350
 	-1   0    0    -1
@@
 	2700 2150 2950 2150
 $Comp
-L Device:Q_PMOS_DGS Q5
+L bldc-BMS:Q_PMOS_6pin Q5
 U 1 1 5BB75D7D
 P 8700 3150
 F 0 "Q5" V 8950 3150 50  0000 C CNN
-F 1 "Q_PMOS_DGS" V 9041 3150 50  0000 C CNN
-F 2 "" H 8900 3250 50  0001 C CNN
+F 1 "Q_PMOS" V 9041 3150 50  0000 C CNN
+F 2 "Package_TO_SOT_SMD:SOT-23-6" H 8900 3250 50  0001 C CNN
 F 3 "~" H 8700 3150 50  0001 C CNN
+F 4 "MOSFET P-CH 60V 4A CPH6" H 0   0   50  0001 C CNN "Description"
+F 5 "CPH6354-TL-WOSCT-ND" H 0   0   50  0001 C CNN "Digikey PN"
 	1    8700 3150
 	0    1    1    0
@@
 F 2 "LED_SMD:LED_0603_1608Metric_Pad1.05x0.95mm_HandSolder" H 7900 5750 50  0001 C CNN
 F 3 "~" H 7900 5750 50  0001 C CNN
+F 4 "LED GREEN CLEAR 0603 SMD	" H 0   0   50  0001 C CNN "Description"
+F 5 "732-4971-1-ND" H 0   0   50  0001 C CNN "Digikey PN"
 	1    7900 5750
 	0    -1   -1   0
