File: Battery Monitor.sch (KiCad schematic (older format))
At the start: 96 parts

Commit message: Updated top-level connections and added MCU
Parts:
- removed C? (x2): 10uF, symbol C_Small
- removed D? (x2): 5.6V, symbol D_Schottky_Small_ALT
- removed Q? (x5): PMOS, symbol Q_DUAL_PNP_PNP_E1B1C2E2B2C1
- removed Q? (x5): PMOS, TO_SOT_Packages_SMD:SOT-666, symbol Q_DUAL_PNP_PNP_E1B1C2E2B2C1
- removed R?: 3.01k, symbol R_Small
- removed R? (x7): 100R, symbol R_Small
- removed R? (x2): 1k, symbol R_Small
- removed R?: 200R, symbol R_Small
- removed TH? (x2): 10k NTC, symbol Thermistor
- added D19: 3.3V, Diode_SMD:D_0603_1608Metric, symbol bldc-BMS-rescue:D_Schottky_Small_ALT
- added D20: 1N4148W, Diode_SMD:D_0603_1608Metric, symbol bldc-BMS-rescue:D_Small_ALT
- added D21: 5.6V, Diode_SMD:D_0603_1608Metric, symbol bldc-BMS-rescue:D_Schottky_Small_ALT
- added J11: Conn_01x07, symbol Connector_Generic:Conn_01x07
- added Q10, Q11, Q12, Q13, Q14, Q15, Q7, Q8, Q9: Q_NMOS_DGS, symbol bldc-BMS-rescue:Q_NMOS_DGS
- added Q6: Q_NMOS_DGS, symbol Device:Q_NMOS_DGS
- added R39: 1k, Resistor_SMD:R_0603_1608Metric, symbol bldc-BMS-rescue:R_Small
- added R51, R52: 10k, Resistor_SMD:R_0603_1608Metric, symbol bldc-BMS-rescue:R_Small
- added R53, R55: 100k, Resistor_SMD:R_0603_1608Metric, symbol bldc-BMS-rescue:R_Small
- added R54, R56: 100R, Resistor_SMD:R_0603_1608Metric, symbol bldc-BMS-rescue:R_Small
- C10: renamed from C?; footprint (none) -> Capacitor_SMD:C_0603_1608Metric; symbol C_Small -> Device:C_Small
- C11, C12, C13, C14, C15, C16, C17, C18, C19, C21, C22, C23, C27: renamed from C?; footprint (none) -> Capacitor_SMD:C_0603_1608Metric; symbol C_Small -> bldc-BMS-rescue:C_Small
- C20: renamed from C?; value C_Small -> 1uF 10V; footprint (none) -> Capacitor_SMD:C_0603_1608Metric; symbol C_Small -> bldc-BMS-rescue:C_Small
- C24: renamed from C?; footprint (none) -> Capacitor_SMD:C_0805_2012Metric; symbol C_Small -> bldc-BMS-rescue:C_Small
- C25, C26: renamed from C?; value 4700pF -> 4.7nF; footprint (none) -> Capacitor_SMD:C_0603_1608Metric; symbol C_Small -> bldc-BMS-rescue:C_Small
- D10, D11, D12, D13, D14, D15, D16, D8, D9: renamed from D?; footprint (none) -> Diode_SMD:D_0603_1608Metric; symbol D_Schottky_Small_ALT -> bldc-BMS-rescue:D_Schottky_Small_ALT
- D17, D22: renamed from D?; value D_Small_ALT -> 1N4148W; footprint (none) -> Diode_SMD:D_0603_1608Metric; symbol D_Small_ALT -> bldc-BMS-rescue:D_Small_ALT
- D18: renamed from D?; value D_Small_ALT -> 1N4148W; footprint (none) -> Diode_SMD:D_0603_1608Metric; symbol D_Small_ALT -> Device:D_Small_ALT
- D7: renamed from D?; footprint (none) -> Diode_SMD:D_0603_1608Metric; symbol D_Schottky_Small_ALT -> Device:D_Schottky_Small_ALT
- J12: renamed from J?; symbol Conn_01x12 -> Connector_Generic:Conn_01x12
- Q16: renamed from Q?; symbol Q_NMOS_DGS -> bldc-BMS-rescue:Q_NMOS_DGS
- R17: renamed from R?; value 100R -> 33R; footprint (none) -> Resistor_SMD:R_1206_3216Metric; symbol R_Small -> Device:R_Small
- R18, R19, R20, R21, R22, R23, R24, R25, R26: renamed from R?; value 100R -> 33R; footprint (none) -> Resistor_SMD:R_1206_3216Metric; symbol R_Small -> bldc-BMS-rescue:R_Small
- R27, R28, R40: renamed from R?; footprint (none) -> Resistor_SMD:R_0603_1608Metric; symbol R_Small -> Device:R_Small
- R29, R30, R31, R32, R33, R34, R35, R36, R37, R38, R41, R42, R43, R44, R45, R46, R47, R48, R49, R57: renamed from R?; footprint (none) -> Resistor_SMD:R_0603_1608Metric; symbol R_Small -> bldc-BMS-rescue:R_Small
- R50: renamed from R?; value 499k -> 100k; footprint (none) -> Resistor_SMD:R_0603_1608Metric; symbol R_Small -> bldc-BMS-rescue:R_Small
- SW1: renamed from SW?; symbol SW_Push -> bldc-BMS-rescue:SW_Push
- U2: renamed from U?; value bq76930 -> bq76930-R1; footprint (none) -> Package_SO:TSSOP-30_4.4x7.8mm_P0.5mm; symbol bq76930 -> bldc-BMS:bq76930-R1
Connections:
- net labels added: BAT, BOOT_RETURN, BOOT_SUPPLY, LOAD+, NTC2, NTC_1, NTC_1_GND, NTC_2_GND, REGSRC, TS1, TS2, VC1, WAKE
- net labels removed: CAP1, VC10X
- wire segments 275 -> 346
Other:
- note added: "10 Cell Configuration"
- note added: "6 Cell Configuration\nC2 == C4\nC7 == C9"
- note added: "BOOT\nAt POR enters SHIP mode."
- note added: "CELL 1"
- note added: "CELL 2"
- note added: "CELL 3"
- note added: "CELL 4"
- note added: "CELL 5"
- note added: "CELL 6\nCELL 5\nCELL 4\nCELL 3\nCELL 2\nCELL 1"
- note added: "Power through balance resistor\nV=IR -> I=V/R = 3.65V/33R = 0.11A\nP=IV -> 0.11A*3.65 = 0.4W"
- note added: "REFERENCE ONLY\nConnectors on first page"
- note added: "REGOUT:\n3.3V NOM 20mA MAX"
- note added: "SHORT"
- note added: "TS1 and TS2:\n10kOHM NTC"
- note removed: "BOOT"
- moved on the sheet: C20, C21, C22, C23, C24, C25, C26, C27, D10, D11, D12, D13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

Commit message: Good-enough for first PCB attempt.
Parts:
- removed C11, C12, C16, C17: 1uF 10V, Capacitor_SMD:C_0603_1608Metric, symbol bldc-BMS-rescue:C_Small
- removed D13, D14, D8, D9: 5.6V, Diode_SMD:D_0603_1608Metric, symbol bldc-BMS-rescue:D_Schottky_Small_ALT
- removed J11: Conn_01x07, symbol Connector_Generic:Conn_01x07
- removed J12: Conn_01x12, symbol Connector_Generic:Conn_01x12
- removed Q10, Q11, Q12, Q13, Q14, Q15, Q7, Q8, Q9: Q_NMOS_DGS, symbol bldc-BMS-rescue:Q_NMOS_DGS
- removed Q6: Q_NMOS_DGS, symbol Device:Q_NMOS_DGS
- removed R18, R19, R23, R24: 33R, Resistor_SMD:R_1206_3216Metric, symbol bldc-BMS-rescue:R_Small
- removed R29, R30, R35, R36: 1k, Resistor_SMD:R_0603_1608Metric, symbol bldc-BMS-rescue:R_Small
- removed R41, R42, R46, R47: 10k, Resistor_SMD:R_0603_1608Metric, symbol bldc-BMS-rescue:R_Small
- added Q10, Q11, Q14, Q15, Q6, Q9: Q_NMOS_GSD, Package_TO_SOT_SMD:SOT-23, symbol Device:Q_NMOS_GSD
- C10, C13, C14, C15, C18, C19, C20, C21: Description (none) -> CAP CER 1UF 25V X5R 0603; Digikey PN (none) -> 1276-1102-1-ND
- C22, C23, C27: value 1uF -> 1uF 10V; Description (none) -> CAP CER 1UF 25V X5R 0603; Digikey PN (none) -> 1276-1102-1-ND
- C24: Description (none) -> CAP CER 4.7UF 25V X5R 0805; Digikey PN (none) -> 1276-1244-1-ND
- C25, C26: Description (none) -> CAP CER 4700PF 50V C0G 0603; Digikey PN (none) -> 445-7400-1-ND
- D10, D11, D12, D15, D16, D21, D7: footprint Diode_SMD:D_0603_1608Metric -> Diode_SMD:D_SOD-323; Description (none) -> Zener Diode 5.6V 400mW ±2% Surface Mount SOD-323; Digikey PN (none) -> MM3Z5V6BCT-ND
- D17, D18, D20, D22: footprint Diode_SMD:D_0603_1608Metric -> Diode_SMD:D_SOD-323; Description (none) -> DIODE GEN PURP 75V 150MA SOD323; Digikey PN (none) -> 1N4148WXTPMSCT-ND
- D19: footprint Diode_SMD:D_0603_1608Metric -> Diode_SMD:D_SOD-323; Description (none) -> TVS DIODE 3.3V SOD323; Digikey PN (none) -> 1727-4152-1-ND
- Q16: value Q_NMOS_DGS -> Q_NMOS_GSD; footprint (none) -> Package_TO_SOT_SMD:SOT-23; symbol bldc-BMS-rescue:Q_NMOS_DGS -> Device:Q_NMOS_GSD; Description (none) -> MOSFET N-CH 20V 0.63A SOT23-3; Digikey PN (none) -> DMN2004KDICT-ND
- R17, R20, R21, R22, R25, R26: footprint Resistor_SMD:R_1206_3216Metric -> Resistor_SMD:R_2010_5025Metric; Description (none) -> RES SMD 33 OHM 5% 3/4W 2010; Digikey PN (none) -> P33WCT-ND
- R27, R28, R31, R32, R33, R34, R37, R38, R39: value 1k -> 1k 1%
- SW1: footprint (none) -> Button_Switch_SMD:SW_SPST_PTS810; Description (none) -> SWITCH TACTILE SPST-NO 50MA 32V; Digikey PN (none) -> CKN10684CT-ND
- U2: value bq76930-R1 -> bq76930; symbol bldc-BMS:bq76930-R1 -> bldc-BMS-rescue:bq76930-R1-bldc-BMS; Description (none) -> IC BATT MGMT LI-ION AFE 30TSSOP; Digikey PN (none) -> 296-39961-1-ND
Connections:
- net labels added: SDA, VC0, VC10, VC4, VC5, VC5B, VC6, VC9
- net labels removed: SCA
- wire segments 346 -> 264
Other:
- note added: "6 Cell Configuration\nSHORT:\nCell 9 (VC8 to VC9)\nCell 8 (VC7 to VC8)\nCell 4 (VC3 to VC4)\nCell 3 (VC2 to VC3)\n\nVC7 == VC9\nVC2 == VC4"
- note added: "CELL 6"
- note added: "REGOUT:\n3.3V nominal, 20mA maximum"
- note added: "Temperature Sensing TS1 and TS2:\n10kOHM NTC"
- note removed: "10 Cell Configuration"
- note removed: "6 Cell Configuration\nC2 == C4\nC7 == C9"
- note removed: "CELL 6\nCELL 5\nCELL 4\nCELL 3\nCELL 2\nCELL 1"
- note removed: "REGOUT:\n3.3V NOM 20mA MAX"
- note removed: "TS1 and TS2:\n10kOHM NTC"
