File: bldc-BMS.kicad_pcb (KiCad board)
At the start: 2 copper layers, 66 x 52.8 mm, 162 parts, among them J1 Conn_01x04, J10 USB_B_Micro, J2 Conn_01x07, J3 Conn_01x02, J5 Conn_01x04, J6 Conn_01x02, J8 Conn_01x06, J9 Conn_01x02, Q2 TBC, Q3 TBC, U1 bq76200, U2 bq76930-R1, U3 BQ78350-R1, U4 AMS1117-3.3, U5 L78L05_SOT89, U6 TJA1042T-3, U7 STM32F072C8, Y1 8MHz

Commit message: Good-enough for first PCB attempt.
Parts:
- removed C17: 1uF 10V, Capacitor_SMD:C_0603_1608Metric
- removed C40, C41: 18pF, Capacitor_SMD:C_0603_1608Metric
- removed D14: 5.6V, Diode_SMD:D_0603_1608Metric
- removed R18, R19, R23, R24: 33R, Resistor_SMD:R_1206_3216Metric
- removed R29, R30, R35, R36: 1k, Resistor_SMD:R_0603_1608Metric
- removed R41, R42, R46, R47: 10k, Resistor_SMD:R_0603_1608Metric
- removed R72: 0R, Resistor_SMD:R_0603_1608Metric
- added D29: D_TVS_x2_AAC, bldc-BMS:D_SOT-23_TVS, F.Cu at (174.6, 56.0)
- added D6: MURS360T3G, Diode_SMD:D_SMC, F.Cu at (169.0, 93.6)
- added JP1: Jumper_NO, Jumper:SolderJumper-2_P1.3mm_Open_TrianglePad1.0x1.5mm, F.Cu at (176.4, 65.2)
- added JP2: Jumper_NO, Jumper:SolderJumper-2_P1.3mm_Open_TrianglePad1.0x1.5mm, F.Cu at (160.2, 51.8)
- added JP3: Jumper_NC_Small, Jumper:SolderJumper-2_P1.3mm_Bridged_RoundedPad1.0x1.5mm, F.Cu at (160.8, 56.4)
- added NT1: Net-Tie, NetTie:NetTie-2_SMD_Pad0.5mm, F.Cu at (115.4, 85.8)
- added Q10: Q_NMOS_GSD, Package_TO_SOT_SMD:SOT-23, F.Cu at (124.0, 52.4)
- added Q11: Q_NMOS_GSD, Package_TO_SOT_SMD:SOT-23, F.Cu at (124.0, 56.4)
- added Q14: Q_NMOS_GSD, Package_TO_SOT_SMD:SOT-23, F.Cu at (124.0, 60.4)
- added Q15: Q_NMOS_GSD, Package_TO_SOT_SMD:SOT-23, F.Cu at (124.0, 64.4)
- added Q16: Q_NMOS_GSD, Package_TO_SOT_SMD:SOT-23, F.Cu at (155.6, 46.8)
- added Q17: ZXMP10A13FTA, Package_TO_SOT_SMD:SOT-23, F.Cu at (149.6, 62.0)
- added Q18: Q_NMOS_GSD, Package_TO_SOT_SMD:SOT-23, F.Cu at (145.8, 69.0)
- added Q5: Q_PMOS, Package_TO_SOT_SMD:SOT-23-6, F.Cu at (139.8, 83.2)
- added Q6: Q_NMOS_GSD, Package_TO_SOT_SMD:SOT-23, F.Cu at (124.0, 44.4)
- added Q9: Q_NMOS_GSD, Package_TO_SOT_SMD:SOT-23, F.Cu at (124.0, 48.4)
- added R7: 100k, Resistor_SMD:R_0603_1608Metric, F.Cu at (155.4, 52.0)
- added R8: 100k, Resistor_SMD:R_0603_1608Metric, F.Cu at (157.0, 52.0)
- added SW1: SW_Push, Button_Switch_SMD:SW_SPST_PTS810, F.Cu at (105.6, 61.2)
- added SW2: SW_Push, Button_Switch_SMD:SW_SPST_PTS810, F.Cu at (159.8, 81.4)
- added TP1: SCL, TestPoint:TestPoint_Pad_D1.5mm, F.Cu at (158.2, 55.0)
- added TP10: BAT-, TestPoint:TestPoint_Pad_D1.5mm, F.Cu at (123.8, 97.2)
- added TP2: SMBC, TestPoint:TestPoint_Pad_D1.5mm, F.Cu at (171.8, 75.2)
- added TP3: REGOUT, TestPoint:TestPoint_Pad_D1.5mm, F.Cu at (120.4, 41.4)
- added TP4: SDA, TestPoint:TestPoint_Pad_D1.5mm, F.Cu at (153.6, 55.0)
- added TP5: SMBD, TestPoint:TestPoint_Pad_D1.5mm, F.Cu at (171.8, 72.6)
- added TP6: BAT+, TestPoint:TestPoint_Pad_D1.5mm, F.Cu at (124.2, 90.4)
- added TP7: LOAD+, TestPoint:TestPoint_Pad_D1.5mm, F.Cu at (162.2, 88.6)
- added TP8: 3.3V, TestPoint:TestPoint_Pad_D1.5mm, F.Cu at (156.8, 59.8)
- added TP9: 5V, TestPoint:TestPoint_Pad_D1.5mm, F.Cu at (173.0, 41.8)
- C11: value 1uF 10V -> 470nF
- C12, C16: value 1uF 10V -> 15pF
- C2, C23, C27: value 1uF -> 1uF 10V
- C22: value 1uF -> 1uF 10V; moved to B.Cu
- C24, C36, R50: moved to B.Cu
- C35, C37, C38: value 2.2uF -> 0.1uF
- C39: value 2.2uF -> 0.1uF; moved to B.Cu
- D10, D11, D12, D15, D16, D17, D18, D19, D2, D20, D21, D22, D3, D7: footprint Diode_SMD:D_0603_1608Metric -> Diode_SMD:D_SOD-323
- D13: value 5.6V -> BLUE; footprint Diode_SMD:D_0603_1608Metric -> LED_SMD:LED_0603_1608Metric_Pad1.05x0.95mm_HandSolder
- D4: footprint Diode_SMD:D_0603_1608Metric -> Diode_SMD:D_SOD-123
- D8: value 5.6V -> RED; footprint Diode_SMD:D_0603_1608Metric -> LED_SMD:LED_0603_1608Metric_Pad1.05x0.95mm_HandSolder
- D9: value 5.6V -> GREEN; footprint Diode_SMD:D_0603_1608Metric -> LED_SMD:LED_0603_1608Metric_Pad1.05x0.95mm_HandSolder
- J1, J5: footprint Connector_JST:JST_PH_B4B-PH-K_1x04_P2.00mm_Vertical -> Connector_JST:JST_PH_S4B-PH-K_1x04_P2.00mm_Horizontal
- J10: footprint Connector_USB:USB_Micro-B_Molex_47346-0001 -> bldc-BMS:USB_Micro-B_Amphenol_10103594-0001LF_Horizontal_circular
- J2: footprint Connector_JST:JST_PH_B7B-PH-K_1x07_P2.00mm_Vertical -> Connector_JST:JST_PH_S7B-PH-K_1x07_P2.00mm_Horizontal
- J3: value Conn_01x02 -> XT60_MALE; footprint bldc-BMS:XT60PW-F -> bldc-BMS:XT60PW-M20
- J6: value Conn_01x02 -> XT60_FEMALE; footprint bldc-BMS:XT60PW-F -> bldc-BMS:XT60PW-F20
- J8: footprint Connector_JST:JST_PH_B6B-PH-K_1x06_P2.00mm_Vertical -> Connector_JST:JST_PH_S6B-PH-K_1x06_P2.00mm_Horizontal
- J9: footprint Connector_JST:JST_PH_B3B-PH-K_1x03_P2.00mm_Vertical -> Connector_JST:JST_PH_S2B-PH-K_1x02_P2.00mm_Horizontal
- Q2, Q3: value TBC -> CSD18531Q5A; footprint Package_SO:PowerPAK_SO-8_Single -> Package_TO_SOT_SMD:TDSON-8-1
- R12, R13, R14: footprint Resistor_SMD:R_0603_1608Metric -> Resistor_SMD:R_1206_3216Metric
- R17, R20, R21, R22, R25, R26: footprint Resistor_SMD:R_1206_3216Metric -> Resistor_SMD:R_2010_5025Metric
- R27, R28, R31, R32, R33, R34, R37, R38, R39: value 1k -> 1k 1%
- R3: footprint Resistor_SMD:R_2816_7142Metric -> Resistor_SMD:R_2512_6332Metric_Pad1.52x3.35mm_HandSolder
- R69, R70: value 510k -> 100k
- R75: value 220R -> 1k
- R76, R77: value 22 -> 22R
- R78: value 120 -> 120R
- U1: footprint Package_SO:HTSSOP-28-1EP_4.4x9.7mm_P0.65mm_EP3.4x9.5mm_ThermalVias -> Package_SO:TSSOP-16_4.4x5mm_P0.65mm
- U2: value bq76930-R1 -> bq76930
- U4: value AMS1117-3.3 -> MIC5219-3.3; footprint Package_TO_SOT_SMD:SOT-223-3_TabPin2 -> bldc-BMS:SOT-23-5
- U5: value L78L05_SOT89 -> MIC5239-5.0; footprint Package_TO_SOT_SMD:SOT-89-3 -> Package_TO_SOT_SMD:SOT-223
- U7: footprint Package_QFP:LQFP-48-1EP_7x7mm_P0.5mm_EP3.6x3.6mm -> Package_QFP:LQFP-48_7x7mm_P0.5mm
- Y1: footprint Oscillator:Oscillator_SMD_Abracon_ASE-4Pin_3.2x2.5mm -> Crystal:Crystal_SMD_5032-4Pin_5.0x3.2mm
- moved C34 97.8 mm to (172.2, 47.8)
- moved C33 89.8 mm to (166.6, 42.6), turned to 270 degrees
- moved C11 84.7 mm to (167.8, 45.8), turned to 180 degrees
- moved C16 81.3 mm to (155.4, 70.4)
- moved D9 79.6 mm to (168.8, 83.4)
- moved D8 78.1 mm to (168.8, 81.6)
- moved C9 76.6 mm to (160.4, 95.4), turned to 270 degrees
- moved D5 76.5 mm to (163.2, 95.4), turned to 90 degrees
- moved D13 76.2 mm to (168.8, 79.8)
- moved C23 75.7 mm to (149.6, 43.2), turned to 270 degrees
- moved C12 74.4 mm to (155.4, 62.6), turned to 180 degrees
- moved C8 73.8 mm to (160.4, 92.2), turned to 270 degrees
- moved J1 70.9 mm to (178.8, 48.6), turned to 90 degrees
- moved R11 70.9 mm to (163.2, 92.0), turned to 270 degrees
- moved D23 67.6 mm to (152.0, 84.2)
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Connections:
- net Net-(C10-Pad1) renamed /Battery Monitor/VC10
- net Net-(C13-Pad2) renamed /Battery Monitor/VC6
- net Net-(C15-Pad1) renamed /Battery Monitor/VC5
- net Net-(C20-Pad2) renamed /Battery Monitor/VC5B
- net Net-(C21-Pad1) renamed /Battery Monitor/VC0
- C10 pad 2: Net-(C10-Pad2) -> /Battery Monitor/VC9
- C11 pad 1: Net-(C10-Pad2) -> Net-(C11-Pad1)
- C11 pad 2: Net-(C10-Pad2) -> GND
- C12 pad 1: Net-(C10-Pad2) -> GND
- C12 pad 2: Net-(C10-Pad2) -> Net-(C12-Pad2)
- C13 pad 1: Net-(C10-Pad2) -> /Battery Monitor/VC9
- C15 pad 2: Net-(C15-Pad2) -> /Battery Monitor/VC4
- C16 pad 1: Net-(C15-Pad2) -> GND
- C16 pad 2: Net-(C15-Pad2) -> Net-(C16-Pad2)
- C18 pad 1: Net-(C15-Pad2) -> /Battery Monitor/VC4
- D1 pad 2: GND -> /Power Stage/BAT-
- D12 pad 2: /Battery Monitor/C4 -> /Battery Monitor/C2
- D13 pad 2: /Battery Monitor/C3 -> +5V
- D7 pad 2: /Battery Monitor/C9 -> /Battery Monitor/C7
- D8 pad 2: /Battery Monitor/C8 -> +5V
- D9 pad 2: /Battery Monitor/C7 -> +5V
- J10 pad 1: (no net) -> Net-(J10-Pad1)
- J2 pad 1: /Battery Monitor/C0 -> /Battery Controller/C10
- J2 pad 2: /Battery Monitor/C1 -> /Battery Monitor/C7
- J2 pad 3: /Battery Monitor/C2 -> /Battery Monitor/C6
- J2 pad 5: /Battery Monitor/C6 -> /Battery Monitor/C2
- J2 pad 6: /Battery Monitor/C7 -> /Battery Monitor/C1
- J2 pad 7: /Battery Controller/C10 -> /Battery Monitor/C0
- J3 pad 1: GND -> /Power Stage/BAT+
- J3 pad 2: /Power Stage/BAT+ -> /Power Stage/BAT-
- Q2 pad 1: Net-(Q2-Pad1) -> /Power Stage/BAT+
- Q2 pad 2: Net-(Q2-Pad2) -> /Power Stage/BAT+
- Q2 pad 4: (no net) -> Net-(Q2-Pad4)
- Q2 pad 5: (no net) -> Net-(Q2-Pad5)
- Q3 pad 1: Net-(Q2-Pad1) -> /Battery Monitor/LOAD+
- Q3 pad 2: Net-(Q3-Pad2) -> /Battery Monitor/LOAD+
- Q3 pad 4: (no net) -> Net-(Q3-Pad4)
- Q3 pad 5: (no net) -> Net-(Q2-Pad5)
- R12 pad 2: Net-(Q2-Pad1) -> Net-(Q2-Pad5)
- R13 pad 2: Net-(Q2-Pad1) -> Net-(Q2-Pad5)
- R14 pad 2: Net-(Q2-Pad1) -> Net-(Q2-Pad5)
- R15 pad 2: (no net) -> Net-(Q5-Pad3)
- R17 pad 1: (no net) -> Net-(Q6-Pad3)
- R2 pad 2: GND -> /Power Stage/BAT-
- R20 pad 1: (no net) -> Net-(Q9-Pad3)
- R21 pad 1: (no net) -> Net-(Q10-Pad3)
- R22 pad 1: (no net) -> Net-(Q11-Pad3)
- R25 pad 1: (no net) -> Net-(Q14-Pad3)
- R26 pad 1: (no net) -> Net-(Q15-Pad3)
- R28 pad 1: Net-(C10-Pad2) -> /Battery Monitor/VC9
- R28 pad 2: /Battery Monitor/C9 -> /Battery Monitor/C7
- R3 pad 1: GND -> /Power Stage/BAT-
- R34 pad 1: Net-(C15-Pad2) -> /Battery Monitor/VC4
- R34 pad 2: /Battery Monitor/C4 -> /Battery Monitor/C2
- R40 pad 2: Net-(C10-Pad2) -> /Battery Monitor/VC9
- R45 pad 1: Net-(C15-Pad2) -> /Battery Monitor/VC4
- R55 pad 1: (no net) -> Net-(Q16-Pad1)
- R56 pad 1: (no net) -> Net-(Q16-Pad2)
- R58 pad 1: (no net) -> Net-(Q17-Pad1)
- R6 pad 2: Net-(Q2-Pad2) -> Net-(Q2-Pad4)
- R61 pad 2: (no net) -> Net-(Q18-Pad3)
- R73 pad 1: (no net) -> Net-(D8-Pad1)
- R74 pad 1: (no net) -> Net-(D9-Pad1)
- R75 pad 1: (no net) -> Net-(D13-Pad1)
- R9 pad 2: Net-(Q3-Pad2) -> Net-(Q3-Pad4)
- U2 pad 17: Net-(C10-Pad2) -> /Battery Monitor/VC9
- U2 pad 18: Net-(C10-Pad2) -> /Battery Monitor/VC9
- U2 pad 19: Net-(C10-Pad2) -> /Battery Monitor/VC9
- U2 pad 23: Net-(C15-Pad2) -> /Battery Monitor/VC4
- U2 pad 24: Net-(C15-Pad2) -> /Battery Monitor/VC4
- U2 pad 25: Net-(C15-Pad2) -> /Battery Monitor/VC4
- U4 pad 1: GND -> +5V
- U4 pad 2: +3V3 -> GND
- U4 pad 3: /Battery Controller/C10 -> +5V
- U5 pad 1: +5V -> /Battery Controller/C10
- U5 pad 3: /Battery Controller/C10 -> +5V
- U7 pad 12: (no net) -> /Battery Controller/~ENABLE
- U7 pad 44: GND -> Net-(JP3-Pad2)
- U7 pad 5: Net-(C40-Pad1) -> Net-(C12-Pad2)
- U7 pad 6: Net-(C41-Pad1) -> Net-(C16-Pad2)
- Y1 pad 1: Net-(C40-Pad1) -> Net-(C12-Pad2)
- Y1 pad 2: Net-(C41-Pad1) -> GND
- Y1 pad 3: (no net) -> Net-(C16-Pad2)
- Y1 pad 4: (no net) -> GND
Routing:
- net /Battery Controller/C10: track 0.00 -> 133.3 mm, vias 0 -> 6
- net /Battery Monitor/NTC_2_GND: track 0.00 -> 92.3 mm, vias 0 -> 2
- net +3V3: track 0.00 -> 88.7 mm, vias 0 -> 5
- net /Battery Monitor/LOAD+: track 19.1 -> 102.9 mm, vias 0 -> 9
- net +5V: track 0.00 -> 83.1 mm, vias 0 -> 2
- net /Battery Controller/REGOUT: track 0.00 -> 75.4 mm, vias 0 -> 5
- net /Battery Monitor/BOOT_SUPPLY: track 0.00 -> 73.3 mm, vias 0 -> 2
- net /Battery Monitor/NTC2: track 0.00 -> 64.4 mm
- net /Battery Monitor/SRP: track 0.00 -> 62.5 mm, vias 0 -> 2
- net /Battery Monitor/NTC_1: track 0.00 -> 62.3 mm, vias 0 -> 2
- net /CAN and USB Interface/I2C1_SCL: track 0.00 -> 61.5 mm, vias 0 -> 2
- net /Battery Monitor/SRN: track 0.00 -> 61.2 mm, vias 0 -> 2
- net /CAN and USB Interface/I2C1_SDA: track 0.00 -> 59.3 mm, vias 0 -> 2
- net /Battery Monitor/WAKE: track 0.00 -> 58.8 mm, vias 0 -> 4
- net /Power Stage/BAT-: track 0.00 -> 55.5 mm, vias 0 -> 9
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- added copper zone on B.Cu, net /Battery Monitor/LOAD+
- added copper zone on F.Cu, net /Battery Monitor/LOAD+
- added copper zone on B.Cu, net /Power Stage/BAT+
- added copper zone on F.Cu, net /Power Stage/BAT+
- added copper zone on B.Cu, net /Power Stage/BAT-
- added copper zone on F.Cu, net /Power Stage/BAT-
- added copper zone on B.Cu, net /Power Stage/LOAD-
- added copper zone on F.Cu, net /Power Stage/LOAD-
- added copper zone on B.Cu, net GND
- added copper zone on F.Cu, net GND
- added copper zone on B.Cu, net Net-(Q2-Pad5)
- added copper zone on F.Cu, net Net-(Q2-Pad5)
Other:
- board size 66 x 52.8 mm -> 82.8 x 63 mm
- net class Default: via_dia 0.8 -> 0.7; via_drill 0.4 -> 0.3
- net class Power added: clearance 0.2, trace_width 0.4, via_dia 0.8, via_drill 0.4
- rule pad_to_mask_clearance: 0.2 -> 0.1
- board text added: "+V BATTERY 0V"
- board text added: "26650 = 26mm x 65mm 2x26mm = 52mm 3x26mm = 69mm"
- board text added: "BATT+"
- board text added: "BATT-"
- board text added: "BATTERY"
- board text added: "Boot"
- board text added: "Display"
- board text added: "LOAD"
- board text added: "bldc-bms 2019-06 MPater"
